File: td2210_reva/td2210_reva.kicad_sch (KiCad schematic)
At the start: 4 parts

Commit message: changes following first build
Parts:
- added Item5 (x2): Conn_01x02, symbol Connector_Generic:Conn_01x02
Connections:
- net Item3: now also Item5.1 (Pin_1), Item5.1 (Pin_1), Item5.2 (Pin_2), Item5.2 (Pin_2); no longer Item2.1 (Pin_1), Item2.10 (Pin_10), Item2.11 (Pin_11), Item2.13 (Pin_13), Item2.14 (Pin_14), Item2.2 (Pin_2), Item2.4 (Pin_4), Item2.5 (Pin_5), Item2.6 (Pin_6), Item2.7 (Pin_7), Item2.8 (Pin_8), Item2.9 (Pin_9)
Other:
- note added: "Assembly Instructions: 1. Equally space the triax connectors centered on the longest side of the box 2. Add Earthing stud to centered short side of the box. 3. Triax chassis connection is shown as GND 4. All connections should be heat shrinked 5. Apply labels for sockets to exterior of box 6. Item 2, supplied inside box 7. Assembly should be labelled with drawing number"
- note added: "Box Label: Force Hi"
- note added: "Box Label: Force/Sense Low"
- note added: "Box Label: Sense Hi"
- note added: "Parts list: 1. Pomona 5219, Triax bulkhead socket, 3 off 2. Pomona 5251, SOIC 14 test clip - 1 off 3. Multicomp 0.5mm^2 flexible cable, 100mm - 4 off 4. Diecast box 115x90x55 - 1 off 5. Header 2.54 single row, 1x2 - 2 off 6. Heat shrink sleeve 1.5mm inner dia recovered, 2cm, Red - 1 off 7. Heat shrink sleeve 1.5mm inner dia recovered, 2cm, Blue - 1 off 8. Heat shrink sleeve 1.5mm inner dia recove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"
- note removed: "Assembly Instructions: 1. Triax chassis connection is shown as GND 2. All connections should be heat shrinked 3. Apply labels for sockets to exterior of box 4. Assembly should be labelled with drawing number"
- note removed: "Label: Force Hi"
- note removed: "Label: Force/Sense Low"
- note removed: "Label: Sense Hi"
- note removed: "Parts list: 1. Pomona 5219, Triax bulkhead socket, 3 off 2. Pomona 5251, SOIC 14 test clip - 1 off 3. Multicomp 0.5mm^2 flexible cable, 100mm - 4 off 4. Diecast box 115x90x55 - 1 off"
- moved on the sheet: Item2
